Commit message: Added support to run on IsaacSim through NVIDIA Brev

File: cone_nav/urdf/f1tenth_base.urdf.xacro (robot description, xacro)
@@ -13,4 +13,5 @@
   </link>
   <link name="zed2i_left_camera_frame"/>
+  <link name="zed2i_left_camera_optical_frame"/>
   <joint name="base_to_zed_left" type="fixed">
     <parent link="base_link"/>
@@ -18,3 +19,9 @@
     <origin xyz="0.20 0.0 0.20" rpy="0 0 0"/>
   </joint>
+  <!-- ROS optical convention: +Z forward, +X right, +Y down. -->
+  <joint name="zed_left_to_optical" type="fixed">
+    <parent link="zed2i_left_camera_frame"/>
+    <child link="zed2i_left_camera_optical_frame"/>
+    <origin xyz="0 0 0" rpy="-1.57079632679 0 -1.57079632679"/>
+  </joint>
 </robot>

Commit message: Added obstacle detection and avoidance

File: cone_nav/urdf/f1tenth_base.urdf.xacro (robot description, xacro)
@@ -14,4 +14,5 @@
   <link name="zed2i_left_camera_frame"/>
   <link name="zed2i_left_camera_optical_frame"/>
+  <link name="zed2i_right_camera_optical_frame"/>
   <joint name="base_to_zed_left" type="fixed">
     <parent link="base_link"/>
@@ -25,3 +26,9 @@
     <origin xyz="0 0 0" rpy="-1.57079632679 0 -1.57079632679"/>
   </joint>
+  <!-- ZED 2i nominal 0.12 m stereo baseline; optical +X points right. -->
+  <joint name="zed_left_optical_to_right_optical" type="fixed">
+    <parent link="zed2i_left_camera_optical_frame"/>
+    <child link="zed2i_right_camera_optical_frame"/>
+    <origin xyz="0.12 0 0" rpy="0 0 0"/>
+  </joint>
 </robot>
